File: 900MHz_Radio_Hardware/demodulator.kicad_sch (KiCad schematic)
At the start: 14 parts, among them Q1 BSS138

Commit message: Worked on demodulator
Connections:
- net GNDPWR: now also U10.23 (COM3), U10.27 (COM1), U10.7 (COM3), U10.9 (COM2)
- net at U10.18 (VDT2): now also U10.6 (IAIN), U10.8 (IMXO)
- net at U10.20 (VDT1): now also U10.22 (QMXO), U10.24 (QAIN)
Other:
- moved on the sheet: C26, C27, R18, TR1
