File: 900MHz_Radio_Hardware/microcontroller.kicad_sch (KiCad schematic)
At the start: 14 parts, among them J1 RJ45_LED_Shielded, SW2 SW_SPDT, U2 Teensy4.1_DEV-16771, U7 MCP4725xxx-xCH

Commit message: Worked on demodulator
Parts:
- added C10: 0.1u, symbol Device:C_Small
- added C35: 10u, symbol Device:C_Small
- U2: footprint MODULE_DEV-16771 -> MRDT_Shields:Teensy_4_1_Ethernet
Connections:
- net +3V3: now also C10.1, C35.1
- net GNDA: now also C10.2, C35.2
Changed lines of the file:
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@@
   (junction (at 229.87 91.44) (diameter 0) (color 0 0 0 0)
   )
+  (junction (at 43.18 162.56) (diameter 0) (color 0 0 0 0)
+  )
   (junction (at 237.49 40.64) (diameter 0) (color 0 0 0 0)
+  )
+  (junction (at 57.15 162.56) (diameter 0) (color 0 0 0 0)
   )
   (junction (at 237.49 33.02) (diameter 0) (color 0 0 0 0)
@@
     (stroke (width 0) (type default))
   )
+  (wire (pts (xy 57.15 168.91) (xy 57.15 171.45))
+    (stroke (width 0) (type default))
+  )
   (wire (pts (xy 245.11 76.2) (xy 245.11 91.44))
     (stroke (width 0) (type default))
@@
     (stroke (width 0) (type default))
   )
-  (wire (pts (xy 43.18 167.64) (xy 43.18 173.99))
+  (wire (pts (xy 43.18 160.02) (xy 43.18 162.56))
     (stroke (width 0) (type default))
   )
@@
     (stroke (width 0) (type default))
   )
+  (wire (pts (xy 64.77 162.56) (xy 64.77 163.83))
+    (stroke (width 0) (type default))
+  )
   (wire (pts (xy 261.62 40.64) (xy 261.62 44.45))
     (stroke (width 0) (type default))
@@
     (stroke (width 0) (type default))
   )
+  (wire (pts (xy 64.77 168.91) (xy 64.77 171.45))
+    (stroke (width 0) (type default))
+  )
   (wire (pts (xy 255.27 15.24) (xy 255.27 13.97))
     (stroke (width 0) (type default))
@@
     (stroke (width 0) (type default))
   )
+  (wire (pts (xy 43.18 162.56) (xy 43.18 173.99))
+    (stroke (width 0) (type default))
+  )
   (wire (pts (xy 264.16 38.1) (xy 264.16 49.53))
     (stroke (width 0) (type default))
@@
     (stroke (width 0) (type default))
   )
+  (wire (pts (xy 43.18 162.56) (xy 57.15 162.56))
+    (stroke (width 0) (type default))
+  )
   (wire (pts (xy 43.18 189.23) (xy 43.18 191.77))
     (stroke (width 0) (type default))
@@
     (stroke (width 0) (type default))
   )
+  (wire (pts (xy 57.15 162.56) (xy 57.15 163.83))
+    (stroke (width 0) (type default))
+  )
   (wire (pts (xy 172.72 88.9) (xy 201.93 88.9))
     (stroke (width 0) (type default))
   )
   (wire (pts (xy 196.85 83.82) (xy 201.93 83.82))
+    (stroke (width 0) (type default))
+  )
+  (wire (pts (xy 64.77 162.56) (xy 57.15 162.56))
     (stroke (width 0) (type default))
   )
@@
     )
   )
+  (symbol (lib_id "Device:C_Small") (at 57.15 166.37 0) (unit 1)
+    (in_bom yes) (on_board yes) (dnp no) (fields_autoplaced)
+    (property "Reference" "C10" (at 59.69 165.1063 0)
+      (effects (font (size 1.27 1.27)) (justify left))
+    )
+    (property "Value" "0.1u" (at 59.69 167.6463 0)
+      (effects (font (size 1.27 1.27)) (justify left))
+    )
+    (property "Footprint" "" (at 57.15 166.37 0)
+      (effects (font (size 1.27 1.27)) hide)
+    )
+    (property "Datasheet" "~" (at 57.15 166.37 0)
+      (effects (font (size 1.27 1.27)) hide)
+    )
+    (pin "1")
+    (pin "2")
+    (instances
+      (project "900MHz_Radio_Hardware"
+        (path "/8d477a51-3dbb-4c04-84c7-90186d141eda/fd7e5d4a-4a71-414e-9993-037c48e39dc4"
+          (reference "C10") (unit 1)
+        )
+      )
+    )
+  )
   (symbol (lib_id "Device:C_Small") (at 233.68 40.64 90) (unit 1)
     (in_bom yes) (on_board yes) (dnp no)
@@
     )
   )
-  (symbol (lib_id "power:+3V3") (at 43.18 167.64 0) (unit 1)
-    (in_bom yes) (on_board yes) (dnp no) (fields_autoplaced)
-    (property "Reference" "#PWR036" (at 43.18 171.45 0)
-      (effects (font (size 1.27 1.27)) hide)
-    )
-    (property "Value" "+3V3" (at 43.18 162.56 0)
-      (effects (font (size 1.27 1.27)))
-    )
-    (property "Footprint" "" (at 43.18 167.64 0)
-      (effects (font (size 1.27 1.27)) hide)
-    )
-    (property "Datasheet" "" (at 43.18 167.64 0)
+  (symbol (lib_id "power:+3V3") (at 43.18 160.02 0) (unit 1)
+    (in_bom yes) (on_board yes) (dnp no) (fields_autoplaced)
+    (property "Reference" "#PWR036" (at 43.18 163.83 0)
+      (effects (font (size 1.27 1.27)) hide)
+    )
+    (property "Value" "+3V3" (at 43.18 154.94 0)
+      (effects (font (size 1.27 1.27)))
+    )
+    (property "Footprint" "" (at 43.18 160.02 0)
+      (effects (font (size 1.27 1.27)) hide)
+    )
+    (property "Datasheet" "" (at 43.18 160.02 0)
       (effects (font (size 1.27 1.27)) hide)
     )
@@
         (path "/8d477a51-3dbb-4c04-84c7-90186d141eda/fd7e5d4a-4a71-414e-9993-037c48e39dc4"
           (reference "#PWR045") (unit 1)
+        )
+      )
+    )
+  )
+  (symbol (lib_id "power:GNDA") (at 57.15 171.45 0) (unit 1)
+    (in_bom yes) (on_board yes) (dnp no) (fields_autoplaced)
+    (property "Reference" "#PWR066" (at 57.15 177.8 0)
+      (effects (font (size 1.27 1.27)) hide)
+    )
+    (property "Value" "GNDA" (at 57.15 176.53 0)
+      (effects (font (size 1.27 1.27)))
+    )
+    (property "Footprint" "" (at 57.15 171.45 0)
+      (effects (font (size 1.27 1.27)) hide)
+    )
+    (property "Datasheet" "" (at 57.15 171.45 0)
+      (effects (font (size 1.27 1.27)) hide)
+    )
+    (pin "1")
+    (instances
+      (project "900MHz_Radio_Hardware"
+        (path "/8d477a51-3dbb-4c04-84c7-90186d141eda/fd7e5d4a-4a71-414e-9993-037c48e39dc4"
+          (reference "#PWR066") (unit 1)
+        )
+      )
+    )
+  )
+  (symbol (lib_id "Device:C_Small") (at 64.77 166.37 0) (unit 1)
+    (in_bom yes) (on_board yes) (dnp no) (fields_autoplaced)
+    (property "Reference" "C35" (at 67.31 165.1063 0)
+      (effects (font (size 1.27 1.27)) (justify left))
+    )
+    (property "Value" "10u" (at 67.31 167.6463 0)
+      (effects (font (size 1.27 1.27)) (justify left))
+    )
+    (property "Footprint" "" (at 64.77 166.37 0)
+      (effects (font (size 1.27 1.27)) hide)
+    )
+    (property "Datasheet" "~" (at 64.77 166.37 0)
+      (effects (font (size 1.27 1.27)) hide)
+    )
+    (pin "1")
+    (pin "2")
+    (instances
+      (project "900MHz_Radio_Hardware"
+        (path "/8d477a51-3dbb-4c04-84c7-90186d141eda/fd7e5d4a-4a71-414e-9993-037c48e39dc4"
+          (reference "C35") (unit 1)
         )
       )
@@
       (effects (font (size 1.27 1.27)))
     )
-    (property "Footprint" "MODULE_DEV-16771" (at 200.66 78.74 0)
+    (property "Footprint" "MRDT_Shields:Teensy_4_1_Ethernet" (at 200.66 78.74 0)
       (effects (font (size 1.27 1.27)) (justify left bottom) hide)
     )
@@
         )
       )
+    )
+  )
+  (symbol (lib_id "power:GNDA") (at 64.77 171.45 0) (unit 1)
+    (in_bom yes) (on_board yes) (dnp no) (fields_autoplaced)
+    (property "Reference" "#PWR067" (at 64.77 177.8 0)
+      (effects (font (size 1.27 1.27)) hide)
+    )
+    (property "Value" "GNDA" (at 64.77 176.53 0)
+      (effects (font (size 1.27 1.27)))
+    )
+    (property "Footprint" "" (at 64.77 171.45 0)
+      (effects (font (size 1.27 1.27)) hide)
+    )
+    (property "Datasheet" "" (at 64.77 171.45 0)
+      (effects (font (size 1.27 1.27)) hide)
+    )
+    (pin "1")
+    (instances
+      (project "900MHz_Radio_Hardware"
+        (path "/8d477a51-3dbb-4c04-84c7-90186d141eda/fd7e5d4a-4a71-414e-9993-037c48e39dc4"
+          (reference "#PWR067") (unit 1)
+        )
+      )
